Commit message: rviz fix

File: gscn_pioneer_description/urdf/common_properties.xacro (robot description, xacro)
@@ -1,28 +1,26 @@
 <?xml version="1.0" ?>
-<!--
-  Various useful properties such as constants and materials
- -->
+<!--  Various useful properties such as constants and materials  -->
 <robot name="xacro_properties" xmlns:xacro="http://ros.org/wiki/xacro">
-  <xacro:property name="M_PI" value="3.1415926535897931" />
-    <material name="White">
-      <color rgba="0.9 0.9 0.9 1"/>
-    </material>
-    <material name="Grey">
-      <color rgba="0.6 0.6 0.6 0.3"/>
-    </material>
-    <material name="Grey_frame">
-      <color rgba="0.6 0.6 0.6 1"/>
-    </material>
-    <material name="Black">
-      <color rgba="0.1 0.1 0.1 1"/>
-    </material>
-    <material name="Red">
-      <color rgba="0.7 0.2 0.1 1"/>
-    </material>
-    <material name="Grey_blue">
-      <color rgba="0.1 0.1 0.3 0.3" />
-    </material>
-    <material name="Orange">
-      <color rgba="1.0 0.4 0.0 1"/>
-    </material>
+	<xacro:property name="M_PI" value="3.1415926535897931" />
+	<material name="White">
+		<color rgba="0.9 0.9 0.9 1"/>
+	</material>
+	<material name="Grey">
+		<color rgba="0.6 0.6 0.6 0.3"/>
+	</material>
+	<material name="Grey_frame">
+		<color rgba="0.6 0.6 0.6 1"/>
+	</material>
+	<material name="Black">
+		<color rgba="0.1 0.1 0.1 1"/>
+	</material>
+	<material name="Red">
+		<color rgba="0.7 0.2 0.1 1"/>
+	</material>
+	<material name="Grey_blue">
+		<color rgba="0.1 0.1 0.3 0.3" />
+	</material>
+	<material name="Orange">
+		<color rgba="1.0 0.4 0.0 1"/>
+	</material>
 </robot>

Commit message: gscn_description: robot visualisation

File: gscn_pioneer_description/urdf/common_properties.xacro (robot description, xacro)
@@ -10,5 +10,5 @@
 	</material>
 	<material name="Grey_frame">
-		<color rgba="0.6 0.6 0.6 1"/>
+		<color rgba="0.2 0.2 0.2 1"/>
 	</material>
 	<material name="Black">

File: gscn_pioneer_description/urdf/pioneer_model.xacro (robot description, xacro)
@@ -7,18 +7,18 @@
 	<link name="frame">
 		<collision>
-			<origin	xyz="0 0 0" rpy="0 0 0" />
+			<origin	xyz="-0.07968 -0.07968 -0.077" rpy="0 0 0" />
 			<geometry>
-				<cylinder radius="0.8" length="0.25"/>
+				<cylinder radius="0.2" length="0.2"/>
 			</geometry>
 		</collision>
 			<visual>
-				<origin	xyz="0 0 0" rpy="${M_PI/2} 0 0" />
+				<origin	xyz="-0.085 -0.085 -0.077" rpy="0 0 0" />
 				<geometry>
-					<mesh filename="package://gscn_pioneer_description/meshes/frame.stl" />
+					<mesh filename="package://gscn_pioneer_description/meshes/pioneer_frame.stl" />
 				</geometry>
-				<material name="Red" />
+				<material name="Grey_frame" />
 			</visual>
 		<inertial>
-			<mass value="1.5"/>
+			<mass value="0.4"/>
 			<inertia 	ixx="0" ixy="0" ixz="0"
 						iyy="0" iyz="0"
@@ -27,9 +27,7 @@
 	</link>
 <!-- Build copter rays -->
-	<ray_stick side="r" num="1" angle="-${M_PI/6}" />
-	<ray_stick side="r" num="2"	angle="-${M_PI/2}" />
-	<ray_stick side="r" num="3" angle="-${M_PI*5/6}" />
-	<ray_stick side="l" num="1"	angle="${M_PI/6}" />
-	<ray_stick side="l" num="2"	angle="${M_PI/2}" />
-	<ray_stick side="l" num="3" angle="${M_PI*5/6}" />
+	<ray_stick side="r" num="1" angle="-${M_PI/4}" />
+	<ray_stick side="r" num="2"	angle="-${M_PI*3/4}" />
+	<ray_stick side="l" num="1"	angle="${M_PI/4}" />
+	<ray_stick side="l" num="2"	angle="${M_PI*3/4}" />
 </robot>

File: gscn_pioneer_description/urdf/pioneer_ray.xacro (robot description, xacro)
@@ -3,81 +3,39 @@
 <!-- Build ray -->
 	<xacro:macro name="ray_stick" params="side num angle">
-  	<joint name="ray_joint_${side}${num}" type="revolute">
-    		<origin xyz="0 0 0" rpy="0 0 ${angle}" />
-    		<parent link="frame" />
-    		<child link="arm_${side}${num}" />
+	<joint name="ray_joint_${side}${num}" type="revolute">
+		<origin xyz="0 0 0" rpy="0 0 ${angle}" />
+		<parent link="frame" />
+		<child link="arm_${side}${num}" />
 		<limit lower="0" upper="0" effort="0" velocity="0" />
-  	</joint>
-    	<link name="arm_${side}${num}">
-		<!--<collision>
-			<origin	xyz="${0.11+0.095} 0 -0.008" rpy="0 0 0" />
-			<geometry>
-				<box size="0.19 0.035 0.055"/>
-			</geometry>
-		</collision>
-    		<visual>
-      			<origin	xyz="0.11 0 0" rpy="0 0 0" />
-    		</visual>-->
+	</joint>
+	<link name="arm_${side}${num}">
 		<inertial>
 			<mass value="0.08"/>
 			<inertia 	ixx="0" ixy="0" ixz="0"
-					iyy="0" iyz="0"
-					izz="0"/>
+						iyy="0" iyz="0"
+						izz="0"/>
 		</inertial>
 	</link>
-  	<joint name="motor_joint_${side}${num}" type="revolute">
-    		<origin xyz="0.535 0 0" rpy="0 0 0" />
-    		<parent link="arm_${side}${num}" />
-    		<child link="motor_${side}${num}" />
+	<joint name="propeller_joint_${side}${num}" type="revolute">
+		<origin xyz="0.095 0 0.017" rpy="0 0 0" />
+		<parent link="arm_${side}${num}" />
+		<child link="propeller_${side}${num}" />
 		<limit lower="0" upper="0" effort="0" velocity="0" />
-  	</joint>
-    	<link name="motor_${side}${num}">
-		<!--<collision>
-			<origin	xyz="0 0 0.03" rpy="0 0 0" />
-			<geometry>
-				<cylinder radius="0.017" length="0.03"/>
-			</geometry>
-		</collision>-->
-    		<visual>
-      			<origin	xyz="0 0 0.03" rpy="0 0 0" />
-      			<geometry>
-				<cylinder radius="0.04" length="0.05"/>
-      			</geometry>
-     			<material name="Orange" />
-    		</visual>
-		<inertial>
-			<mass value="0.055"/>
-			<inertia 	ixx="0" ixy="0" ixz="0"
-					iyy="0" iyz="0"
-					izz="0"/>
-		</inertial>
-	</link>
-  	<joint name="propeller_joint_${side}${num}" type="revolute">
-    		<origin xyz="0 0 0.055" rpy="0 0 0" />
-    		<parent link="motor_${side}${num}" />
-    		<child link="propeller_${side}${num}" />
-    		<limit lower="0" upper="0" effort="0" velocity="0" />
-  	</joint>
-    	<link name="propeller_${side}${num}">
-		<!--<collision>
+	</joint>
+	<link name="propeller_${side}${num}">
+		<visual>
 			<origin	xyz="0 0 0" rpy="0 0 0" />
 			<geometry>
-				<cylinder radius="0.11" length="0.015"/>
+				<cylinder radius="0.06" length="0.006"/>
 			</geometry>
-		</collision>-->
-    		<visual>
-      			<origin	xyz="0 0 0" rpy="0 0 0" />
-      			<geometry>
-				<cylinder radius="0.18" length="0.015"/>
-      			</geometry>
-     			<material name="Grey" />
-    		</visual>
+			<material name="Grey" />
+		</visual>
 		<inertial>
 			<mass value="0.015"/>
 			<inertia 	ixx="0" ixy="0" ixz="0"
-					iyy="0" iyz="0"
-					izz="0"/>
+						iyy="0" iyz="0"
+						izz="0"/>
 		</inertial>
 	</link>
-	</xacro:macro>
+</xacro:macro>
 </robot>
