Commit message: lidar changes

File: gscn_pioneer_description/urdf/pioneer_model.xacro (robot description, xacro)
@@ -5,5 +5,5 @@
 	<xacro:include filename="$(find gscn_pioneer_description)/urdf/common_properties.xacro"/>
 <!-- Build the body frame -->
-	<link name="frame">
+	<link name="base_link">
 		<collision>
 			<origin	xyz="-0.07968 -0.07968 -0.077" rpy="0 0 0" />
@@ -17,5 +17,5 @@
 					<mesh filename="package://gscn_pioneer_description/meshes/pioneer_frame.stl" />
 				</geometry>
-				<material name="Grey_frame" />
+				<material name="White" />
 			</visual>
 		<inertial>

File: gscn_pioneer_description/urdf/pioneer_ray.xacro (robot description, xacro)
@@ -3,7 +3,7 @@
 <!-- Build ray -->
 	<xacro:macro name="ray_stick" params="side num angle">
-	<joint name="ray_joint_${side}${num}" type="revolute">
+	<joint name="ray_joint_${side}${num}" type="fixed">
 		<origin xyz="0 0 0" rpy="0 0 ${angle}" />
-		<parent link="frame" />
+		<parent link="base_link" />
 		<child link="arm_${side}${num}" />
 		<limit lower="0" upper="0" effort="0" velocity="0" />
@@ -17,5 +17,5 @@
 		</inertial>
 	</link>
-	<joint name="propeller_joint_${side}${num}" type="revolute">
+	<joint name="propeller_joint_${side}${num}" type="fixed">
 		<origin xyz="0.095 0 0.017" rpy="0 0 0" />
 		<parent link="arm_${side}${num}" />
